File: HM-RC-8_Remote/HM-RC-8_Remote-v01-008.sch (EAGLE design)
At the start: 18 parts, among them M2 ARDUINO-PRO-MINI-3.3V#NP

Commit message: Remote
Parts:
- removed RAW: (no value), jumper:SJ
- removed X5: (no value), adafruit:SMACONNECTOR_EDGE
- added J1: (no value), SparkFun-Connectors:CONN_02PTH3
- added JP1: JUMPER-SMT_3_1-NC_TRACE_SILK, SparkFun-Jumpers:JUMPER-SMT_3_1-NC_TRACE_SILK
Connections:
- removed net N$10: 8.2
- removed net N$6: 4.2
- removed net N$7: 5.2
- removed net N$8: 6.2
- removed net N$9: 7.2
- removed net UREG: RAW.2
- new net N$4: J1.1, JP1.2
- net 16-A2: now also 7.2
- net 17-A3: now also 8.2
- net ANT0: no longer X5.ANT
- net D6: now also 6.2
- net D7: now also 4.2
- net D9: now also 5.2
- net GND: now also J1.2; no longer X5.GND1, X5.GND2, X5.GND3, X5.GND4
- net RAW: no longer RAW.1
- net VCC: now also JP1.3
- net VIN: now also JP1.1
Other:
- moved on the sheet: C3
