File: HM-RC-8_Remote/HM-RC-8_Remote-v03-019.brd (EAGLE design)
At the start: 65 x 24 mm, 18 parts, among them M2 ARDUINO-PRO-MINI-3.3V#NP, SW1 SW-TACTILE-TL3305, SW2 SW-TACTILE-TL3305, SW3 SW-TACTILE-TL3305, SW4 SW-TACTILE-TL3305, SW5 SW-TACTILE-TL3305, SW6 SW-TACTILE-TL3305, SW7 SW-TACTILE-TL3305, SW8 SW-TACTILE-TL3305

Commit message: V03, Pics
Parts:
- removed ICLUSION: DTSM-3, mechanics:DTSM-3
- removed M2: ARDUINO-PRO-MINI-3.3V#NP, diy-modules-Martin:ARDUINO-PRO-MINI#NP
- added M1: ARDUINO-PRO-MINI-#MARTIN-REMOTE, diy-modules-Martin:ARDUINO-PRO-MINI#NP-MARTIN-REMOTE
- added SW9: SW-TACTILE-TL3305, we-switch:TL3305
- moved ANT 12.6 mm to (60.7, 24.0)
- moved CC0 2.96 mm to (40.4, 14.5), turned to 150 degrees
- moved C3 2.00 mm to (27.9, 2.44)
- moved C5 2.00 mm to (19.1, 2.44)
- moved L1 2.00 mm to (11.4, 2.44)
- moved STEPUP 2.00 mm to (15.2, 2.44)
- moved SW2 2.00 mm to (10.2, 2.44)
- moved SW4 2.00 mm to (25.4, 2.44)
- moved SW6 2.00 mm to (40.6, 2.44)
- moved SW8 2.00 mm to (55.9, 2.44)
- moved J1 2.00 mm to (2.54, 9.43)
- moved JP1 2.00 mm to (6.35, 1.81)
- moved SW1 2.00 mm to (10.2, 19.0)
- moved SW3 2.00 mm to (25.4, 19.0)
- moved SW5 2.00 mm to (40.6, 19.0)
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Connections:
- removed net A5: M2.J3.1
- removed net A6: M2.J3.2
- removed net A7: M2.J3.3
- removed net N$1: M2.J6.2
- removed net N$3: SW2.1, SW2.4
- net 14-A0: now also M1.A0; no longer M2.J6.8
- net 15-A1: now also M1.A1; no longer M2.J6.7
- net 16-A2: now also M1.A2; no longer M2.J6.6
- net 17-A3: now also M1.A3; no longer M2.J6.5
- net CSN: now also M1.10; no longer M2.J6.12
- net D3: now also M1.3; no longer M2.J7.7
- net D4: now also M1.4; no longer M2.J7.6
- net D5: now also M1.5; no longer M2.J7.5
- net D6: now also M1.6; no longer M2.J7.4
- net D7: now also M1.7; no longer M2.J7.3
- net D8: now also M1.8, SW9.2, SW9.3; no longer ICLUSION.2, M2.J7.2
- net D9: now also M1.9; no longer M2.J7.1
- net GND: now also M1.GND, M1.GND2, SW2.1, SW2.4, SW9.1, SW9.4; no longer ICLUSION.1, M2.J7.9
- net IRQ: now also M1.2; no longer M2.J7.8
- net MISO: now also M1.12; no longer M2.J6.10
- net MOSI: now also M1.11; no longer M2.J6.11
- net RAW: now also M1.RAW; no longer M2.J6.1
- net RESET: now also M1.RST1; no longer M2.J7.10
- net RX: now also M1.RX; no longer M2.J7.11
- net SCK: now also M1.13; no longer M2.J6.9
- net TX: now also M1.TX; no longer M2.J7.12
- net VCC: now also M1.VCC; no longer M2.J6.4
Routing:
- net GND: track 157.9 -> 244.4 mm, vias 23 -> 28
- net D9: track 89.4 -> 42.5 mm
- net D8: track 58.9 -> 34.2 mm, vias 1 -> 0
- net VCC: track 76.5 -> 92.7 mm
- net IRQ: track 34.0 -> 19.7 mm, vias 0 -> 1
- net MOSI: track 41.4 -> 50.6 mm, vias 0 -> 1
- net MISO: track 43.5 -> 37.0 mm, vias 1 -> 2
- net N$3: track 6.40 -> 0.00 mm
- net ANT0: track 1.87 -> 7.69 mm
- net 17-A3: track 47.2 -> 52.9 mm
- net 16-A2: track 42.9 -> 38.0 mm
- net 15-A1: track 14.2 -> 10.0 mm
- net D6: track 34.9 -> 30.9 mm
- net D7: track 22.2 -> 18.2 mm
- net 14-A0: track 8.07 -> 10.9 mm
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Other:
- board size 65 x 24 mm -> 65 x 26 mm
- board text added: "86mm"
- board text added: "Ant"
- board text added: "HM-Remote V0.3 www.neuby.de"
- board text added: "TX"
- board text added: "optional"
- board text removed: "HM-Remote V0.2 www.neuby.de"
