File: HM-RC-8_Remote/HM-RC-8_Remote-v03-019.sch (EAGLE design)
At the start: 18 parts, among them M2 ARDUINO-PRO-MINI-3.3V#NP, SW1 SW-TACTILE-TL3305, SW2 SW-TACTILE-TL3305, SW3 SW-TACTILE-TL3305, SW4 SW-TACTILE-TL3305, SW5 SW-TACTILE-TL3305, SW6 SW-TACTILE-TL3305, SW7 SW-TACTILE-TL3305, SW8 SW-TACTILE-TL3305

Commit message: V03, Pics
Parts:
- removed ICLUSION: DTSM-3, mechanics:DTSM-3
- removed M2: ARDUINO-PRO-MINI-3.3V#NP, diy-modules-Martin:ARDUINO-PRO-MINI-3.3V#NP
- added M1: ARDUINO-PRO-MINI-#MARTIN-REMOTE, diy-modules-Martin:ARDUINO-PRO-MINI-#MARTIN-REMOTE
- added SW9: SW-TACTILE-TL3305, we-switch:SW-TACTILE-TL3305
Connections:
- removed net A5: M2.GND.3
- removed net A6: M2.A6
- removed net A7: M2.A7
- removed net N$1: M2.GND.2
- removed net N$3: SW2.P1
- net 14-A0: now also M1.A0; no longer M2.A0
- net 15-A1: now also M1.A1; no longer M2.A1
- net 16-A2: now also M1.A2; no longer M2.A2
- net 17-A3: now also M1.A3; no longer M2.A3
- net CSN: now also M1.D10; no longer M2.D10
- net D3: now also M1.D3; no longer M2.D3
- net D4: now also M1.D4; no longer M2.D4
- net D5: now also M1.D5; no longer M2.D5
- net D6: now also M1.D6; no longer M2.D6
- net D7: now also M1.D7; no longer M2.D7
- net D8: now also M1.D8, SW9.S1; no longer ICLUSION.2, M2.D8
- net D9: now also M1.D9; no longer M2.D9
- net GND: now also M1.GND.1, M1.GND.2, SW2.P1, SW9.P1; no longer ICLUSION.1, M2.GND.1
- net IRQ: now also M1.D2; no longer M2.D2
- net MISO: now also M1.D12; no longer M2.D12
- net MOSI: now also M1.D11; no longer M2.D11
- net RAW: now also M1.RAW; no longer M2.RAW
- net RESET: now also M1.RST.2; no longer M2.RST.2
- net RX: now also M1.D0/RX; no longer M2.D0/RX
- net SCK: now also M1.D13; no longer M2.D13
- net TX: now also M1.D1/TX; no longer M2.D1/TX
- net VCC: now also M1.VCC; no longer M2.VCC
Other:
- note added: "button 4*4*1.5"
- note removed: "Achtung nur wenn physikalisch an der Position von GND.3 der A5 Pin ist verbinden !!!"
